File: shmoergh-dual-rail-psu.kicad_sch (KiCad schematic)
At the start: 43 parts, among them J1 Screw_Terminal_01x02, J2 Screw_Terminal_01x03, J3 Screw_Terminal_01x02, Q1 AO3401A, Q2 AO3401A, U1 TPS5430DDA, U2 TPS65131RGER

Commit message: Component update
Parts:
- removed H2, H4: MountingHole, MountingHole:MountingHole_3mm_Pad_Via, symbol Mechanical:MountingHole
- U2: LCSC TPS65131RGER -> C87663
Connections:
- net +12V: now also J2.3 (Pin_3); no longer J2.1 (Pin_1)
- net -12V: now also J2.1 (Pin_1); no longer J2.3 (Pin_3)
- net GND: now also J1.1 (Pin_1), U2.25 (PGND_TH); no longer J1.2 (Pin_2)
- net VIN: now also J1.2 (Pin_2); no longer J1.1 (Pin_1)
- net C1: now reaches C1.1, Q1.2 (S), U1.7 (VIN)
Other:
- note added: "VoutN = -12.1V"
- note removed: "VoutP = -12.1V"
- moved on the sheet: J2
Changed lines of the file:
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@@
+    (stroke (width 0) (type default))
+  )
+  (wire (pts (xy 71.12 171.45) (xy 69.85 171.45))
     (stroke (width 0) (type default))
   )
@@
   )
   (wire (pts (xy 74.93 78.74) (xy 74.93 80.01))
+    (stroke (width 0) (type default))
+  )
+  (wire (pts (xy 69.85 171.45) (xy 69.85 173.99))
     (stroke (width 0) (type default))
   )
@@
     (effects (font (size 1.27 1.27) (thickness 0.254) bold) (justify left bottom))
   )
-  (text "VoutP = -12.1V" (at 148.59 154.94 0)
+  (text "VoutN = -12.1V" (at 148.59 154.94 0)
     (effects (font (size 1.27 1.27)) (justify left bottom))
   )
@@
   )
   (label "OUTN" (at 115.57 161.29 0) (fields_autoplaced)
+    (effects (font (size 1.27 1.27)) (justify left bottom))
+  )
+  (label "C1" (at 50.8 60.96 0) (fields_autoplaced)
     (effects (font (size 1.27 1.27)) (justify left bottom))
   )
@@
     )
   )
-  (symbol (lib_id "Mechanical:MountingHole") (at 234.95 158.75 0) (unit 1)
-    (in_bom no) (on_board yes) (dnp no) (fields_autoplaced)
-    (property "Reference" "H4" (at 237.49 157.48 0)
-      (effects (font (size 1.27 1.27)) (justify left))
-    )
-    (property "Value" "MountingHole" (at 237.49 160.02 0)
-      (effects (font (size 1.27 1.27)) (justify left))
-    )
-    (property "Footprint" "MountingHole:MountingHole_3mm_Pad_Via" (at 234.95 158.75 0)
-      (effects (font (size 1.27 1.27)) hide)
-    )
-    (property "Datasheet" "~" (at 234.95 158.75 0)
-      (effects (font (size 1.27 1.27)) hide)
-    )
-    (instances
-      (project "shmoergh-dual-rail-psu"
-        (path "/89d328a3-7e80-44bd-8c4d-7128e2c0b3c8"
-          (reference "H4") (unit 1)
-        )
-      )
-    )
-  )
   (symbol (lib_id "Diode:B340") (at 106.68 72.39 270) (unit 1)
     (in_bom yes) (on_board yes) (dnp no) (fields_autoplaced)
@@
       (effects (font (size 1.27 1.27)) hide)
     )
-    (property "LCSC" "TPS65131RGER" (at 87.63 151.13 0)
+    (property "LCSC" "C87663" (at 87.63 151.13 0)
       (effects (font (size 1.27 1.27)))
     )
@@
     (pin "23")
     (pin "24")
+    (pin "25")
     (pin "3")
     (pin "4")
@@
     )
   )
-  (symbol (lib_id "Connector:Screw_Terminal_01x03") (at 222.25 128.27 0) (mirror y) (unit 1)
+  (symbol (lib_id "Connector:Screw_Terminal_01x03") (at 222.25 128.27 180) (unit 1)
     (in_bom no) (on_board yes) (dnp no)
-    (property "Reference" "J2" (at 222.25 133.35 0)
-      (effects (font (size 1.27 1.27)))
-    )
-    (property "Value" "Screw_Terminal_01x03" (at 222.25 121.92 0)
+    (property "Reference" "J2" (at 222.25 123.19 0)
+      (effects (font (size 1.27 1.27)))
+    )
+    (property "Value" "Screw_Terminal_01x03" (at 222.25 120.65 0)
       (effects (font (size 1.27 1.27)))
     )
@@
     )
   )
-  (symbol (lib_id "Connector:Screw_Terminal_01x02") (at 196.85 125.73 0) (unit 1)
+  (symbol (lib_id "Connector:Screw_Terminal_01x02") (at 196.85 128.27 0) (mirror x) (unit 1)
     (in_bom no) (on_board yes) (dnp no)
-    (property "Reference" "J1" (at 196.85 134.62 0)
+    (property "Reference" "J1" (at 196.85 119.38 0)
       (effects (font (size 1.27 1.27)))
     )
@@
       (effects (font (size 1.27 1.27)))
     )
-    (property "Footprint" "TerminalBlock_Phoenix:TerminalBlock_Phoenix_MKDS-1,5-2_1x02_P5.00mm_Horizontal" (at 196.85 125.73 0)
-      (effects (font (size 1.27 1.27)) hide)
-    )
-    (property "Datasheet" "~" (at 196.85 125.73 0)
+    (property "Footprint" "TerminalBlock_Phoenix:TerminalBlock_Phoenix_MKDS-1,5-2_1x02_P5.00mm_Horizontal" (at 196.85 128.27 0)
+      (effects (font (size 1.27 1.27)) hide)
+    )
+    (property "Datasheet" "~" (at 196.85 128.27 0)
       (effects (font (size 1.27 1.27)) hide)
     )
@@
         )
       )
-    )
-  )
-  (symbol (lib_id "Mechanical:MountingHole") (at 198.12 158.75 0) (unit 1)
-    (in_bom no) (on_board yes) (dnp no) (fields_autoplaced)
-    (property "Reference" "H2" (at 200.66 157.48 0)
-      (effects (font (size 1.27 1.27)) (justify left))
-    )
-    (property "Value" "MountingHole" (at 200.66 160.02 0)
-      (effects (font (size 1.27 1.27)) (justify left))
-    )
-    (property "Footprint" "MountingHole:MountingHole_3mm_Pad_Via" (at 198.12 158.75 0)
-      (effects (font (size 1.27 1.27)) hide)
-    )
-    (property "Datasheet" "~" (at 198.12 158.75 0)
-      (effects (font (size 1.27 1.27)) hide)
-    )
-    (instances
-      (project "shmoergh-dual-rail-psu"
-        (path "/89d328a3-7e80-44bd-8c4d-7128e2c0b3c8"
-          (reference "H2") (unit 1)
-        )
-      )
